Commit message: Full bringup: cmd_vel relay, RViz config, Docker/DDS fixes, TF completeness
- Add cmd_vel_relay.py: bridges /cmd_vel (Twist) → ackermann reference (TwistStamped)
- Add RViz config generated from within RViz (hand-written configs break Orbit mouse input)
- Switch to Cyclone DDS on loopback (cyclonedds.xml) — Fast-DDS multicast fails across
  Docker containers even with --network host
- Makefile: all secondary targets (rviz, teleop, shell) use docker exec into named picar2
  container; bringup adds --network host, --ipc host, xhost, X11 socket
- Export position state interfaces for passive front wheel joints so joint_state_broadcaster
  publishes complete TF tree (no more missing frame errors in RViz)
- Dockerfile: add teleop-twist-keyboard and rmw-cyclonedds-cpp

Co-Authored-By: Claude Sonnet 4.6 <noreply@anthropic.com>

File: src/picar2_description/urdf/picar2.urdf.xacro (robot description, xacro)
@@ -40,4 +40,11 @@
       <state_interface name="position"/>
     </joint>
+    <!-- Front wheels — passive (no encoder); position held at 0 for TF -->
+    <joint name="front_left_wheel_joint">
+      <state_interface name="position"/>
+    </joint>
+    <joint name="front_right_wheel_joint">
+      <state_interface name="position"/>
+    </joint>
   </ros2_control>
   <!-- ═══════════════════════════════════════════════════

Commit message: lidar: stable scan orientation via blind-spot gap detection
The LDS02RR has no fixed angular reference — index 0xA0 lands at a
random rotor position each motor start. Fix: detect the 3 consistently
missing indices (motor blind spot) each revolution and use their centre
as a hardware reference, placing it at π (behind robot). This makes
scan orientation repeatable across restarts without any hardware change.

Also fix packet sync: on checksum/index failure, back up 1 byte instead
of discarding the full 22-byte window, preventing false-0xFA misalignment.

URDF: remove erroneous 180° yaw on laser_joint (reset to 0); update Z
position to measured value. angle_offset parameter remains for
mounting-angle fine-tune on top of auto-calibration.

Co-Authored-By: Claude Sonnet 4.6 <noreply@anthropic.com>

File: src/picar2_description/urdf/picar2.urdf.xacro (robot description, xacro)
@@ -251,5 +251,5 @@
   <!-- Sensors (fixed) -->
   <joint name="laser_joint" type="fixed">
-    <origin xyz="0.012548 0 0.1311" rpy="0 0 3.1416"/>
+    <origin xyz="0.012548 0 0.147" rpy="0 0 0"/>
     <parent link="base_link"/>
     <child  link="laser_link"/>

Commit message: imu: axis remapping, mounting-tilt correction, gyro/accel calibration support
- Remap chip axes (chip Y→robot X, -X→robot Y) in dispatch_imu_frame
- Apply mounting-tilt rotation matrix (Ry(pitch)*Rx(roll)) to accel,
  gyro, and mag so Madgwick sees (0,0,g) when robot is flat
- Read imu_mount_roll / imu_mount_pitch from URDF <hardware> params;
  precompute rotation matrix in on_init() — update params after imu cal accel
- URDF: add imu_mount_roll=-0.1648 / imu_mount_pitch=-0.0657 params;
  set base_imu joint rpy="0 0 0" (correction now done in driver)
- Disable magnetometer (soft-iron distortion from motors causes drift)

Co-Authored-By: Claude Sonnet 4.6 <noreply@anthropic.com>

File: src/picar2_description/urdf/picar2.urdf.xacro (robot description, xacro)
@@ -12,4 +12,7 @@
       <param name="port">$(arg port)</param>
       <param name="baud">$(arg baud)</param>
+      <!-- IMU mounting tilt (rad) — re-run `imu cal accel` and update if IMU is remounted -->
+      <param name="imu_mount_roll">-0.1648</param>
+      <param name="imu_mount_pitch">-0.0657</param>
     </hardware>
     <!-- Rear drive wheels (velocity-controlled) -->
@@ -206,5 +209,5 @@
     <parent link="base_link"/>
     <child  link="imu_link"/>
-    <origin xyz="-0.05 0.0 0.05" rpy="0 3.1415 1.5707"/>
+    <origin xyz="-0.05 0.0 0.05" rpy="0 0 0"/>
   </joint>
   <!-- Rear wheels (continuous — drive wheels) -->

Commit message: sim: add Gazebo Harmonic simulation support
- URDF: use_sim xacro arg switches hardware plugin between
  picar2_control/Picar2Hardware (real) and gz_ros2_control/GazeboSimSystem;
  adds gz_ros2_control plugin, IMU + GPU LiDAR Gazebo sensors, primitive
  collision shapes (box/cylinder), wheel friction, joint damping
- sim.launch.py: launches Gazebo with room.sdf, spawns robot, bridges
  sensors to ROS, runs same controllers/EKF/relay as real robot
- worlds/room.sdf: 5×5 m walled room with two obstacles for SLAM/nav testing
- gz_bridge.yaml: bridges /imu/data_raw, /scan, /clock from Gazebo to ROS
- Dockerfile: adds ros-jazzy-ros-gz-sim, ros-gz-bridge, gz-ros2-control
- Makefile: adds `make sim` target (container named picar2 — slam/nav/teleop work unchanged)

Workflow: make sim → make cartographer → make nav → 2D Nav Goal in RViz

Co-Authored-By: Claude Sonnet 4.6 <noreply@anthropic.com>

File: src/picar2_description/urdf/picar2.urdf.xacro (robot description, xacro)
@@ -1,6 +1,7 @@
 <?xml version="1.0" encoding="utf-8"?>
 <robot name="picar2" xmlns:xacro="http://ros.org/wiki/xacro">
-  <xacro:arg name="port" default="/dev/ttyYahboom0"/>
-  <xacro:arg name="baud" default="460800"/>
+  <xacro:arg name="port"    default="/dev/ttyYahboom0"/>
+  <xacro:arg name="baud"    default="460800"/>
+  <xacro:arg name="use_sim" default="false"/>
   <!-- ═══════════════════════════════════════════════════
        ros2_control block — joint names match URDF joints
@@ -9,13 +10,18 @@
   <ros2_control name="picar2" type="system">
     <hardware>
-      <plugin>picar2_control/Picar2Hardware</plugin>
-      <param name="port">$(arg port)</param>
-      <param name="baud">$(arg baud)</param>
-      <!-- IMU mounting tilt (rad) — re-run `imu cal accel` and update if IMU is remounted -->
-      <param name="imu_mount_roll">-0.1648</param>
-      <param name="imu_mount_pitch">-0.0657</param>
-      <!-- Steering: µs per radian for servo0. Default: (max_pulse-min_pulse)/2 / max_steer_rad
-           = (2025-885)/2 / 0.6 = 950. Tune with circle test to correct servo linkage error. -->
-      <param name="steer_us_per_rad">1020.0</param>
+      <xacro:if value="$(arg use_sim)">
+        <plugin>gz_ros2_control/GazeboSimSystem</plugin>
+      </xacro:if>
+      <xacro:unless value="$(arg use_sim)">
+        <plugin>picar2_control/Picar2Hardware</plugin>
+        <param name="port">$(arg port)</param>
+        <param name="baud">$(arg baud)</param>
+        <!-- IMU mounting tilt (rad) — re-run `imu cal accel` and update if IMU is remounted -->
+        <param name="imu_mount_roll">-0.1648</param>
+        <param name="imu_mount_pitch">-0.0657</param>
+        <!-- Steering: µs per radian for servo0. Default: (max_pulse-min_pulse)/2 / max_steer_rad
+             = (2025-885)/2 / 0.6 = 950. Tune with circle test to correct servo linkage error. -->
+        <param name="steer_us_per_rad">1020.0</param>
+      </xacro:unless>
     </hardware>
     <!-- Rear drive wheels (velocity-controlled) -->
@@ -54,4 +60,13 @@
     </joint>
   </ros2_control>
+  <!-- Gazebo: gz_ros2_control plugin (sim only) -->
+  <xacro:if value="$(arg use_sim)">
+    <gazebo>
+      <plugin filename="gz_ros2_control-system"
+              name="gz_ros2_control::GazeboSimROS2ControlPlugin">
+        <parameters>$(find picar2_bringup)/config/controllers.yaml</parameters>
+      </plugin>
+    </gazebo>
+  </xacro:if>
   <!-- ═══════════════════════════════════════════════════
        Links
@@ -73,6 +88,6 @@
     </visual>
     <collision>
-      <origin xyz="0 0 0" rpy="0 0 0"/>
-      <geometry><mesh filename="package://picar2_description/meshes/base_link.STL"/></geometry>
+      <origin xyz="0 0 0.04" rpy="0 0 0"/>
+      <geometry><box size="0.24 0.17 0.08"/></geometry>
     </collision>
   </link>
@@ -91,6 +106,6 @@
     </visual>
     <collision>
-      <origin xyz="0 0 0" rpy="0 0 0"/>
-      <geometry><mesh filename="package://picar2_description/meshes/back_right_link.STL"/></geometry>
+      <origin xyz="0 0 0" rpy="1.5708 0 0"/>
+      <geometry><cylinder radius="0.033" length="0.025"/></geometry>
     </collision>
   </link>
@@ -109,6 +124,6 @@
     </visual>
     <collision>
-      <origin xyz="0 0 0" rpy="0 0 0"/>
-      <geometry><mesh filename="package://picar2_description/meshes/back_right_link.STL"/></geometry>
+      <origin xyz="0 0 0" rpy="1.5708 0 0"/>
+      <geometry><cylinder radius="0.033" length="0.025"/></geometry>
     </collision>
   </link>
@@ -127,6 +142,6 @@
     </visual>
     <collision>
-      <origin xyz="0 0 0" rpy="0 0 0"/>
-      <geometry><mesh filename="package://picar2_description/meshes/front_left_steer.STL"/></geometry>
+      <origin xyz="0 0 -0.01" rpy="0 0 0"/>
+      <geometry><box size="0.02 0.02 0.03"/></geometry>
     </collision>
   </link>
@@ -145,6 +160,6 @@
     </visual>
     <collision>
-      <origin xyz="0 0 0" rpy="0 0 0"/>
-      <geometry><mesh filename="package://picar2_description/meshes/back_right_link.STL"/></geometry>
+      <origin xyz="0 0 0" rpy="1.5708 0 0"/>
+      <geometry><cylinder radius="0.033" length="0.025"/></geometry>
     </collision>
   </link>
@@ -163,6 +178,6 @@
     </visual>
     <collision>
-      <origin xyz="0 0 0" rpy="0 0 0"/>
-      <geometry><mesh filename="package://picar2_description/meshes/front_left_steer.STL"/></geometry>
+      <origin xyz="0 0 -0.01" rpy="0 0 0"/>
+      <geometry><box size="0.02 0.02 0.03"/></geometry>
     </collision>
   </link>
@@ -181,6 +196,6 @@
     </visual>
     <collision>
-      <origin xyz="0 0 0" rpy="0 0 0"/>
-      <geometry><mesh filename="package://picar2_description/meshes/back_right_link.STL"/></geometry>
+      <origin xyz="0 0 0" rpy="1.5708 0 0"/>
+      <geometry><cylinder radius="0.033" length="0.025"/></geometry>
     </collision>
   </link>
@@ -198,5 +213,5 @@
     <collision>
       <origin xyz="0 0 0" rpy="0 0 0"/>
-      <geometry><mesh filename="package://picar2_description/meshes/laser_link.STL"/></geometry>
+      <geometry><box size="0.07 0.07 0.05"/></geometry>
     </collision>
   </link>
@@ -220,4 +235,5 @@
     <child  link="back_right_link"/>
     <axis xyz="0 1 0"/>
+    <dynamics damping="0.01" friction="0.0"/>
   </joint>
   <joint name="back_left_joint" type="continuous">
@@ -226,4 +242,5 @@
     <child  link="back_left_link"/>
     <axis xyz="0 1 0"/>
+    <dynamics damping="0.01" friction="0.0"/>
   </joint>
   <!-- Front steering knuckles (revolute — single servo via linkage) -->
@@ -234,4 +251,5 @@
     <axis xyz="0 0 1"/>
     <limit lower="-0.6" upper="0.6" effort="10" velocity="1"/>
+    <dynamics damping="0.01" friction="0.0"/>
   </joint>
   <joint name="front_right_steer_joint" type="revolute">
@@ -241,4 +259,5 @@
     <axis xyz="0 0 1"/>
     <limit lower="-0.6" upper="0.6" effort="10" velocity="1"/>
+    <dynamics damping="0.01" friction="0.0"/>
   </joint>
   <!-- Front wheels (passive — follow steer knuckle) -->
@@ -248,4 +267,5 @@
     <child  link="front_left_wheel"/>
     <axis xyz="0 -1 0"/>
+    <dynamics damping="0.01" friction="0.0"/>
   </joint>
   <joint name="front_right_wheel_joint" type="continuous">
@@ -254,4 +274,5 @@
     <child  link="front_right_wheel"/>
     <axis xyz="0 1 0"/>
+    <dynamics damping="0.01" friction="0.0"/>
   </joint>
   <!-- Sensors (fixed) -->
@@ -261,3 +282,71 @@
     <child  link="laser_link"/>
   </joint>
+  <!-- ═══════════════════════════════════════════════════
+       Gazebo properties (sim only)
+       ═══════════════════════════════════════════════════ -->
+  <!-- Drive wheel friction -->
+  <gazebo reference="back_left_link">
+    <mu1>1.0</mu1><mu2>1.0</mu2>
+    <kp>1e6</kp><kd>1.0</kd>
+  </gazebo>
+  <gazebo reference="back_right_link">
+    <mu1>1.0</mu1><mu2>1.0</mu2>
+    <kp>1e6</kp><kd>1.0</kd>
+  </gazebo>
+  <!-- Front wheels low friction (steered, not driven) -->
+  <gazebo reference="front_left_wheel">
+    <mu1>0.5</mu1><mu2>0.5</mu2>
+  </gazebo>
+  <gazebo reference="front_right_wheel">
+    <mu1>0.5</mu1><mu2>0.5</mu2>
+  </gazebo>
+  <!-- IMU sensor -->
+  <gazebo reference="imu_link">
+    <sensor name="imu_sensor" type="imu">
+      <always_on>1</always_on>
+      <update_rate>50</update_rate>
+      <topic>/model/picar2/imu</topic>
+      <gz_frame_id>imu_link</gz_frame_id>
+      <imu>
+        <angular_velocity>
+          <x><noise type="gaussian"><mean>0</mean><stddev>0.009</stddev></noise></x>
+          <y><noise type="gaussian"><mean>0</mean><stddev>0.009</stddev></noise></y>
+          <z><noise type="gaussian"><mean>0</mean><stddev>0.009</stddev></noise></z>
+        </angular_velocity>
+        <linear_acceleration>
+          <x><noise type="gaussian"><mean>0</mean><stddev>0.021</stddev></noise></x>
+          <y><noise type="gaussian"><mean>0</mean><stddev>0.021</stddev></noise></y>
+          <z><noise type="gaussian"><mean>0</mean><stddev>0.021</stddev></noise></z>
+        </linear_acceleration>
+      </imu>
+    </sensor>
+  </gazebo>
+  <!-- LiDAR sensor -->
+  <gazebo reference="laser_link">
+    <sensor name="lidar" type="gpu_lidar">
+      <always_on>1</always_on>
+      <update_rate>10</update_rate>
+      <topic>/model/picar2/scan</topic>
+      <gz_frame_id>laser_link</gz_frame_id>
+      <lidar>
+        <scan>
+          <horizontal>
+            <samples>360</samples>
+            <resolution>1</resolution>
+            <min_angle>-3.14159265</min_angle>
+            <max_angle>3.14159265</max_angle>
+          </horizontal>
+        </scan>
+        <range>
+          <min>0.06</min>
+          <max>5.0</max>
+          <resolution>0.001</resolution>
+        </range>
+        <noise type="gaussian">
+          <mean>0.0</mean>
+          <stddev>0.01</stddev>
+        </noise>
+      </lidar>
+    </sensor>
+  </gazebo>
 </robot>

Commit message: description: switch laser_link mesh and frame per lidar model
- Add ld19.STL (mm→m scale 0.001) for LD19 lidar visual
- Conditional laser_joint Z rotation: -90° for ld19, 0 for others
- Pass lidar arg through xacro so mesh/frame match the active lidar

Co-Authored-By: Claude Sonnet 4.6 <noreply@anthropic.com>

File: src/picar2_description/urdf/picar2.urdf.xacro (robot description, xacro)
@@ -4,4 +4,6 @@
   <xacro:arg name="baud"    default="460800"/>
   <xacro:arg name="use_sim" default="false"/>
+  <xacro:arg name="lidar"   default="lds02rr"/>
+  <xacro:property name="lidar_model" value="$(arg lidar)"/>
   <!-- ═══════════════════════════════════════════════════
        ros2_control block — joint names match URDF joints
@@ -205,9 +207,18 @@
       <inertia ixx="0" ixy="0" ixz="0" iyy="0" iyz="0" izz="0"/>
     </inertial>
-    <visual>
-      <origin xyz="0 0 0" rpy="0 0 0"/>
-      <geometry><mesh filename="package://picar2_description/meshes/laser_link.STL"/></geometry>
-      <material name=""><color rgba="1 1 1 1"/></material>
-    </visual>
+    <xacro:if value="${lidar_model == 'ld19'}">
+      <visual>
+        <origin xyz="0 0 -0.047" rpy="0 0 -1.5708"/>
+        <geometry><mesh filename="package://picar2_description/meshes/ld19.STL" scale="0.001 0.001 0.001"/></geometry>
+        <material name=""><color rgba="0.2 0.2 0.2 1"/></material>
+      </visual>
+    </xacro:if>
+    <xacro:unless value="${lidar_model == 'ld19'}">
+      <visual>
+        <origin xyz="0 0 0" rpy="0 0 0"/>
+        <geometry><mesh filename="package://picar2_description/meshes/laser_link.STL"/></geometry>
+        <material name=""><color rgba="1 1 1 1"/></material>
+      </visual>
+    </xacro:unless>
     <collision>
       <origin xyz="0 0 0" rpy="0 0 0"/>
