Commit message: picar2: add LD07 as fixed front depth sensor
- URDF: ld07_link + ld07_joint at (0.172, 0, 0.034) m from base_link,
  visualised with ld07_ros_model.stl (mm units, orientation pre-applied,
  rpy="0 0 0" on both joint and visual — ld07_link +X points forward)
- bringup: ldrobot_ld07_node always launched, publishes /ld07/scan in
  ld07_link frame via /dev/ld07 udev symlink
- lidar arg: removed 'ld07' option (sensor is now always-on)
- Makefile: lidar-ld07-view opens RViz with ld07_link fixed frame

Co-Authored-By: Claude Sonnet 4.6 <noreply@anthropic.com>

File: picar2_description/urdf/picar2.urdf.xacro (robot description, xacro)
@@ -226,4 +226,24 @@
     </collision>
   </link>
+  <!-- LD07 structured-light depth sensor — front centre, fixed mount -->
+  <link name="ld07_link">
+    <inertial>
+      <origin xyz="0 0 0" rpy="0 0 0"/>
+      <mass value="0"/>
+      <inertia ixx="0" ixy="0" ixz="0" iyy="0" iyz="0" izz="0"/>
+    </inertial>
+    <visual>
+      <origin xyz="0 0 0" rpy="0 0 0"/>
+      <geometry>
+        <mesh filename="package://picar2_description/meshes/ld07_ros_model.stl"
+              scale="0.001 0.001 0.001"/>
+      </geometry>
+      <material name=""><color rgba="0.15 0.15 0.15 1"/></material>
+    </visual>
+    <collision>
+      <origin xyz="0.015 0 0" rpy="0 0 0"/>
+      <geometry><box size="0.03 0.03 0.015"/></geometry>
+    </collision>
+  </link>
   <!-- ═══════════════════════════════════════════════════
        Joints
@@ -291,4 +311,10 @@
     <parent link="base_link"/>
     <child  link="laser_link"/>
+  </joint>
+  <joint name="ld07_joint" type="fixed">
+    <!-- Front centre, 40 mm above base_link. Tune xyz once mounted. -->
+    <origin xyz="0.172 0 0.034" rpy="0 0 0"/>
+    <parent link="base_link"/>
+    <child  link="ld07_link"/>
   </joint>
   <!-- ═══════════════════════════════════════════════════

Commit message: description: tilt ld07_joint 16° nose-up, sync Gazebo sensor params
Co-Authored-By: Claude Sonnet 4.6 <noreply@anthropic.com>

File: picar2_description/urdf/picar2.urdf.xacro (robot description, xacro)
@@ -5,5 +5,6 @@
   <xacro:arg name="use_sim" default="false"/>
   <xacro:arg name="lidar"   default="lds02rr"/>
-  <xacro:property name="lidar_model" value="$(arg lidar)"/>
+  <xacro:property name="lidar_model"    value="$(arg lidar)"/>
+  <xacro:property name="ld07_tilt_rad"  value="0.2793"/>  <!-- 16° mount angle -->
   <!-- ═══════════════════════════════════════════════════
        ros2_control block — joint names match URDF joints
@@ -234,5 +235,5 @@
     </inertial>
     <visual>
-      <origin xyz="0 0 0" rpy="0 0 0"/>
+      <origin xyz="0 0 0" rpy="0 -${ld07_tilt_rad} 0"/>
       <geometry>
         <mesh filename="package://picar2_description/meshes/ld07_ros_model.stl"
@@ -313,6 +314,5 @@
   </joint>
   <joint name="ld07_joint" type="fixed">
-    <!-- Front centre, 40 mm above base_link. Tune xyz once mounted. -->
-    <origin xyz="0.172 0 0.034" rpy="0 0 0"/>
+    <origin xyz="0.172 0 0.034" rpy="0 ${ld07_tilt_rad} 0"/>
     <parent link="base_link"/>
     <child  link="ld07_link"/>
@@ -370,5 +370,5 @@
             <samples>160</samples>
             <resolution>1</resolution>
-            <min_angle>-0.7854</min_angle>
+            <min_angle>-0.7330</min_angle>
             <max_angle>0.7854</max_angle>
           </horizontal>
@@ -376,5 +376,5 @@
         <range>
           <min>0.005</min>
-          <max>0.170</max>
+          <max>0.400</max>
           <resolution>0.001</resolution>
         </range>

Commit message: description: adjust laser_link position and LD19 visual alignment
Move laser_joint 20 mm down (z: 0.147 → 0.127) so scans match actual
obstacle height. Raise LD19 mesh visual 20 mm (z: -0.047 → -0.027)
to keep the 3D model aligned with the physical sensor.

Co-Authored-By: Claude Sonnet 4.6 <noreply@anthropic.com>

File: picar2_description/urdf/picar2.urdf.xacro (robot description, xacro)
@@ -210,5 +210,5 @@
     <xacro:if value="${lidar_model == 'ld19'}">
       <visual>
-        <origin xyz="0 0 -0.047" rpy="0 0 -1.5708"/>
+        <origin xyz="0 0 -0.027" rpy="0 0 -1.5708"/>
         <geometry><mesh filename="package://picar2_description/meshes/ld19.STL" scale="0.001 0.001 0.001"/></geometry>
         <material name=""><color rgba="0.2 0.2 0.2 1"/></material>
@@ -309,5 +309,5 @@
   <!-- Sensors (fixed) -->
   <joint name="laser_joint" type="fixed">
-    <origin xyz="0.012548 0 0.147" rpy="0 0 0"/>
+    <origin xyz="0.012548 0 0.127" rpy="0 0 0"/>
     <parent link="base_link"/>
     <child  link="laser_link"/>

Commit message: description/bringup: center base_footprint on rear axle
Ackermann navigation requires base_footprint at the rear axle.
Shift base_joint x: 0.0 → 0.11607 m (rear axle distance) so
base_footprint aligns with the drive axle. All child joints are
unchanged — they are relative to base_link, which moves with it.

Update nav2.yaml footprint polygon accordingly:
  old (chassis centre): [[-0.12, 0.12] × [-0.09, 0.09]]
  new (rear axle):      [[-0.04, 0.24] × [-0.09, 0.09]]

Co-Authored-By: Claude Sonnet 4.6 <noreply@anthropic.com>

File: picar2_description/urdf/picar2.urdf.xacro (robot description, xacro)
@@ -253,5 +253,5 @@
     <parent link="base_footprint"/>
     <child  link="base_link"/>
-    <origin xyz="0.0 0.0 0.0215" rpy="0 0 0"/>
+    <origin xyz="0.11607 0.0 0.0215" rpy="0 0 0"/>
   </joint>
   <joint name="base_imu" type="fixed">

Commit message: bringup: add SEN0628 ToF sensor as front sensor
- URDF: add sen0628_link at same mount position as ld07_link (0.172m fwd,
  0.034m up, 16° tilt)
- picar2.launch.py: add SEN0628 lifecycle node (auto configure+activate),
  new use_sen0628/sen0628_port args; flip use_ld07 default to false
- nav2.yaml: replace ld07 LaserScan source with sen0628 PointCloud2 source
  on /sen0628/pointcloud in both local and global costmaps

Co-Authored-By: Claude Sonnet 4.6 <noreply@anthropic.com>

File: picar2_description/urdf/picar2.urdf.xacro (robot description, xacro)
@@ -318,4 +318,11 @@
     <child  link="ld07_link"/>
   </joint>
+  <!-- SEN0628 matrix ToF sensor — same mount position as LD07, no tilt -->
+  <link name="sen0628_link"/>
+  <joint name="sen0628_joint" type="fixed">
+    <origin xyz="0.172 0 0.034" rpy="0 0 0"/>
+    <parent link="base_link"/>
+    <child  link="sen0628_link"/>
+  </joint>
   <!-- ═══════════════════════════════════════════════════
        Gazebo properties (sim only)

Commit message: sim: add SEN0628 ToF sensor to Gazebo model
Co-Authored-By: Claude Sonnet 4.6 <noreply@anthropic.com>

File: picar2_description/urdf/picar2.urdf.xacro (robot description, xacro)
@@ -321,5 +321,5 @@
   <link name="sen0628_link"/>
   <joint name="sen0628_joint" type="fixed">
-    <origin xyz="0.172 0 0.034" rpy="0 0 0"/>
+    <origin xyz="0.172 0 0.034" rpy="${pi} 0 0"/>
     <parent link="base_link"/>
     <child  link="sen0628_link"/>
@@ -377,4 +377,29 @@
         <z><noise type="gaussian"><mean>0.0</mean><stddev>0.0001</stddev></noise></z>
       </magnetometer>
+    </sensor>
+  </gazebo>
+  <!-- SEN0628 8×8 matrix ToF — depth_camera, 45°×45° FOV, 4 m range -->
+  <gazebo reference="sen0628_link">
+    <sensor name="sen0628" type="depth_camera">
+      <always_on>1</always_on>
+      <update_rate>10</update_rate>
+      <topic>/model/picar2/sen0628</topic>
+      <gz_frame_id>sen0628_link</gz_frame_id>
+      <camera>
+        <horizontal_fov>0.7854</horizontal_fov>
+        <image>
+          <width>8</width>
+          <height>8</height>
+        </image>
+        <clip>
+          <near>0.005</near>
+          <far>4.0</far>
+        </clip>
+        <noise>
+          <type>gaussian</type>
+          <mean>0.0</mean>
+          <stddev>0.005</stddev>
+        </noise>
+      </camera>
     </sensor>
   </gazebo>

Commit message: urdf: fix sensor mounts for sen0628 and ld19
sen0628: correct orientation (was upside-down, rpy π→0) and height (z 0.034→0.054 m)

laser_joint: make model-specific — ld19 gets x+30 mm, y+5 mm, yaw+3°;
lds02rr keeps original pose

Co-Authored-By: Claude Sonnet 4.6 <noreply@anthropic.com>

File: picar2_description/urdf/picar2.urdf.xacro (robot description, xacro)
@@ -309,5 +309,10 @@
   <!-- Sensors (fixed) -->
   <joint name="laser_joint" type="fixed">
-    <origin xyz="0.012548 0 0.127" rpy="0 0 0"/>
+    <xacro:if value="${lidar_model == 'ld19'}">
+      <origin xyz="0.042548 0.005 0.127" rpy="0 0 0.0523605"/>
+    </xacro:if>
+    <xacro:unless value="${lidar_model == 'ld19'}">
+      <origin xyz="0.012548 0 0.127" rpy="0 0 0"/>
+    </xacro:unless>
     <parent link="base_link"/>
     <child  link="laser_link"/>
@@ -321,5 +326,5 @@
   <link name="sen0628_link"/>
   <joint name="sen0628_joint" type="fixed">
-    <origin xyz="0.172 0 0.034" rpy="${pi} 0 0"/>
+    <origin xyz="0.172 0 0.054" rpy="0 0 0"/>
     <parent link="base_link"/>
     <child  link="sen0628_link"/>

Commit message: pan/tilt: add ros2_control integration and forward_command_controller
- URDF: add pan_link/tilt_link geometry and pan_joint/tilt_joint
  (revolute, xyz 0.25 0 0.075 from base, tilt 0.03 0 0.04 from pan)
  with position command+state interfaces in ros2_control block;
  pan_us_per_rad/tilt_us_per_rad hardware params (default 500 µs/rad)
- picar2_hardware: export pan/tilt position state+command interfaces;
  write() sends MSG_SERVO_WRITE (0x87) for servo1/servo2 each cycle;
  read() echoes commanded position as state (open-loop); on_deactivate
  sends neutral for both servos
- controllers.yaml: add pan_tilt_controller (ForwardCommandController
  on pan_joint + tilt_joint position interfaces)
- picar2.launch.py + sim.launch.py: spawn pan_tilt_controller

Co-Authored-By: Claude Sonnet 4.6 <noreply@anthropic.com>

File: picar2_description/urdf/picar2.urdf.xacro (robot description, xacro)
@@ -25,4 +25,6 @@
         <param name="steer_lut_us">-595 -454 -410 -364 -329 -299 -271 -252 -202 -151 -121 -101 128 154	193	257	308	354	433	464	493	545</param>
         <param name="steer_lut_rad">0.6756 0.5308 0.4578 0.4058 0.3513 0.3176 0.2790 0.2443 0.1994 0.1392 0.1062 0.0668 -0.1276 -0.1646 -0.2049 -0.2829	-0.3129	-0.3681	-0.4680	-0.4844	-0.5078	-0.6109</param>
+        <param name="pan_us_per_rad">500.0</param>
+        <param name="tilt_us_per_rad">500.0</param>
       </xacro:unless>
     </hardware>
@@ -59,4 +61,19 @@
     </joint>
     <joint name="front_right_wheel_joint">
+      <state_interface name="position"/>
+    </joint>
+    <!-- Pan/tilt servos (servo1=pan, servo2=tilt); open-loop: state = last command -->
+    <joint name="pan_joint">
+      <command_interface name="position">
+        <param name="min">-1.57</param>
+        <param name="max">1.57</param>
+      </command_interface>
+      <state_interface name="position"/>
+    </joint>
+    <joint name="tilt_joint">
+      <command_interface name="position">
+        <param name="min">-1.57</param>
+        <param name="max">1.57</param>
+      </command_interface>
       <state_interface name="position"/>
     </joint>
@@ -329,4 +346,51 @@
     <parent link="base_link"/>
     <child  link="sen0628_link"/>
+  </joint>
+  <!-- Pan/tilt camera mount (servo1=pan, servo2=tilt) -->
+  <link name="pan_link">
+    <inertial>
+      <origin xyz="0 0 0" rpy="0 0 0"/>
+      <mass value="0.02"/>
+      <inertia ixx="1e-06" ixy="0" ixz="0" iyy="1e-06" iyz="0" izz="1e-06"/>
+    </inertial>
+    <visual>
+      <origin xyz="0 0 0" rpy="0 0 0"/>
+      <geometry><box size="0.03 0.03 0.02"/></geometry>
+      <material name=""><color rgba="0.3 0.3 0.3 1"/></material>
+    </visual>
+    <collision>
+      <origin xyz="0 0 0" rpy="0 0 0"/>
+      <geometry><box size="0.03 0.03 0.02"/></geometry>
+    </collision>
+  </link>
+  <link name="tilt_link">
+    <inertial>
+      <origin xyz="0 0 0" rpy="0 0 0"/>
+      <mass value="0.02"/>
+      <inertia ixx="1e-06" ixy="0" ixz="0" iyy="1e-06" iyz="0" izz="1e-06"/>
+    </inertial>
+    <visual>
+      <origin xyz="0 0 0" rpy="0 0 0"/>
+      <geometry><box size="0.03 0.02 0.03"/></geometry>
+      <material name=""><color rgba="0.3 0.3 0.3 1"/></material>
+    </visual>
+    <collision>
+      <origin xyz="0 0 0" rpy="0 0 0"/>
+      <geometry><box size="0.03 0.02 0.03"/></geometry>
+    </collision>
+  </link>
+  <joint name="pan_joint" type="revolute">
+    <origin xyz="0.14 0 0.065" rpy="0 0 0"/>
+    <parent link="base_link"/>
+    <child  link="pan_link"/>
+    <axis xyz="0 0 1"/>
+    <limit lower="-1.57" upper="1.57" effort="1" velocity="1"/>
+  </joint>
+  <joint name="tilt_joint" type="revolute">
+    <origin xyz="0.03 0 0.03" rpy="0 0 0"/>
+    <parent link="pan_link"/>
+    <child  link="tilt_link"/>
+    <axis xyz="0 1 0"/>
+    <limit lower="-1.57" upper="1.57" effort="1" velocity="1"/>
   </joint>
   <!-- ═══════════════════════════════════════════════════

Commit message: sim: add spawn yaw/z, params overlay and ground-truth odometry
Benchmark enablers, all backwards compatible. spawn_yaw could not be set at
all, so any scenario needing a start heading was impossible; spawn_z replaces a
hardcoded 5 cm drop. params_overlay layers a second file over nav2.yaml so a
config variant is a short file instead of a forked 234-line copy.

The xacro gains a sim-only gz odometry publisher for ground truth — the
/world/<w>/pose/info route cannot work, as entity identity lives in pose.name
while the ros_gz Pose_V->TFMessage converter reads header.data — and a
sensor_noise multiplier, since Gazebo exposes no RNG seed.

Co-Authored-By: Claude Opus 5 <noreply@anthropic.com>
Claude-Session: https://claude.ai/code/session_01J91VAG6GU24wcgM3mWkjsN

File: picar2_description/urdf/picar2.urdf.xacro (robot description, xacro)
@@ -5,4 +5,11 @@
   <xacro:arg name="use_sim" default="false"/>
   <xacro:arg name="lidar"   default="lds02rr"/>
+  <!-- Scales every simulated sensor noise stddev. Gazebo Harmonic exposes no
+       RNG seed, so sensor noise is the one source of run-to-run variance that
+       cannot be seeded away. sensor_noise:=0.0 removes it entirely, which turns
+       "how repeatable is this benchmark?" into two measurable questions:
+       variance from physics/sensing vs variance from scheduling. -->
+  <xacro:arg name="sensor_noise" default="1.0"/>
+  <xacro:property name="noise_scale" value="$(arg sensor_noise)"/>
   <xacro:property name="lidar_model"    value="$(arg lidar)"/>
   <xacro:property name="ld07_tilt_rad"  value="0.2793"/>  <!-- 16° mount angle -->
@@ -86,4 +93,19 @@
         <parameters>$(find picar2_bringup)/config/controllers.yaml</parameters>
       </plugin>
+      <!-- Ground-truth pose for the navigation benchmark. Simulation only, so
+           the real robot is unaffected. This exists because the ground truth
+           cannot be obtained from /world/<w>/pose/info: the entity name lives
+           in pose.name, while the ros_gz Pose_V->TFMessage converter reads
+           header.data, so every bridged transform comes out with an empty
+           frame_id. A model-side odometry publisher names its frames
+           explicitly instead. -->
+      <plugin filename="gz-sim-odometry-publisher-system"
+              name="gz::sim::systems::OdometryPublisher">
+        <odom_frame>gt_odom</odom_frame>
+        <robot_base_frame>base_footprint</robot_base_frame>
+        <odom_publish_frequency>50</odom_publish_frequency>
+        <odom_topic>model/picar2/gt_odom</odom_topic>
+        <dimensions>3</dimensions>
+      </plugin>
     </gazebo>
   </xacro:if>
@@ -422,12 +444,12 @@
       <imu>
         <angular_velocity>
-          <x><noise type="gaussian"><mean>0</mean><stddev>0.009</stddev></noise></x>
-          <y><noise type="gaussian"><mean>0</mean><stddev>0.009</stddev></noise></y>
-          <z><noise type="gaussian"><mean>0</mean><stddev>0.009</stddev></noise></z>
+          <x><noise type="gaussian"><mean>0</mean><stddev>${0.009 * noise_scale}</stddev></noise></x>
+          <y><noise type="gaussian"><mean>0</mean><stddev>${0.009 * noise_scale}</stddev></noise></y>
+          <z><noise type="gaussian"><mean>0</mean><stddev>${0.009 * noise_scale}</stddev></noise></z>
         </angular_velocity>
         <linear_acceleration>
-          <x><noise type="gaussian"><mean>0</mean><stddev>0.021</stddev></noise></x>
-          <y><noise type="gaussian"><mean>0</mean><stddev>0.021</stddev></noise></y>
-          <z><noise type="gaussian"><mean>0</mean><stddev>0.021</stddev></noise></z>
+          <x><noise type="gaussian"><mean>0</mean><stddev>${0.021 * noise_scale}</stddev></noise></x>
+          <y><noise type="gaussian"><mean>0</mean><stddev>${0.021 * noise_scale}</stddev></noise></y>
+          <z><noise type="gaussian"><mean>0</mean><stddev>${0.021 * noise_scale}</stddev></noise></z>
         </linear_acceleration>
       </imu>
@@ -442,7 +464,7 @@
       <gz_frame_id>imu_link</gz_frame_id>
       <magnetometer>
-        <x><noise type="gaussian"><mean>0.0</mean><stddev>0.0001</stddev></noise></x>
-        <y><noise type="gaussian"><mean>0.0</mean><stddev>0.0001</stddev></noise></y>
-        <z><noise type="gaussian"><mean>0.0</mean><stddev>0.0001</stddev></noise></z>
+        <x><noise type="gaussian"><mean>0.0</mean><stddev>${0.0001 * noise_scale}</stddev></noise></x>
+        <y><noise type="gaussian"><mean>0.0</mean><stddev>${0.0001 * noise_scale}</stddev></noise></y>
+        <z><noise type="gaussian"><mean>0.0</mean><stddev>${0.0001 * noise_scale}</stddev></noise></z>
       </magnetometer>
     </sensor>
@@ -468,5 +490,5 @@
           <type>gaussian</type>
           <mean>0.0</mean>
-          <stddev>0.005</stddev>
+          <stddev>${0.005 * noise_scale}</stddev>
         </noise>
       </camera>
@@ -496,5 +518,5 @@
         <noise type="gaussian">
           <mean>0.0</mean>
-          <stddev>0.002</stddev>
+          <stddev>${0.002 * noise_scale}</stddev>
         </noise>
       </lidar>
@@ -524,5 +546,5 @@
         <noise type="gaussian">
           <mean>0.0</mean>
-          <stddev>0.01</stddev>
+          <stddev>${0.01 * noise_scale}</stddev>
         </noise>
       </lidar>

Commit message: description: unmirror the front-left wheel axis
The joint used axis (0 -1 0) while the other three wheels use (0 1 0), and the
hardware negated its position estimate to cancel that out. The pair only looked
right because both were wrong, and in simulation - where nothing does the
negating - /joint_states showed the front-left wheel turning backwards as the
robot drove forwards: measured over one run, back_left +117.3 rad and
front_right +64.4 rad against front_left -34.6 rad.

Both now agree, and the same run reports +48.5 and +44.7 rad for the two front
wheels instead of -34.6 and +64.4.

Visualisation only: the joint is passive and state-only, front_left_wheel has
no child links, and odometry comes from the rear wheels and the steer joints.
corner_left is unchanged over three runs (0 reversals, detour 0.991-0.997,
10.2-11.1 s against a 10.53 s baseline). Needs a rebuild on the Pi to reach the
robot, since picar2_control is C++.

Not the cause of the left/right turn asymmetry: both front wheels still roll
about 1.5 m over a 3.3 m path while the rears roll 3.7 m, so they are scrubbing
rather than rolling, and that is still to be explained.

Co-Authored-By: Claude Opus 5 <noreply@anthropic.com>
Claude-Session: https://claude.ai/code/session_01J91VAG6GU24wcgM3mWkjsN

File: picar2_description/urdf/picar2.urdf.xacro (robot description, xacro)
@@ -336,5 +336,12 @@
     <parent link="front_left_steer"/>
     <child  link="front_left_wheel"/>
-    <axis xyz="0 -1 0"/>
+    <!-- +y like every other wheel. This was -y, so the joint reported the
+         front-left wheel turning backwards while the robot drove forwards:
+         measured over one run, back_left +117.3 rad and front_right +64.4 rad
+         against front_left -34.6 rad. Only the reported state and the visual
+         were affected - the collision is a plain cylinder and the joint is
+         passive, state-only - but it made /joint_states describe a robot that
+         cannot exist. -->
+    <axis xyz="0 1 0"/>
     <dynamics damping="0.01" friction="0.0"/>
   </joint>

Commit message: sim: make the front axle roll instead of scrub
Three sim-only defects, all found by watching the wheels in Gazebo.
steering_joints_names was left-first while steering_kinematics.cpp returns
{alpha_r, alpha_l}, so inner and outer steering angles landed on the wrong
wheels. Front joint damping of 0.01 demanded more torque than friction can
supply, so the wheels slid rather than rolled: front rolling 42% -> 84-91%
of rear. And the front wheel bottoms sat 0.4 mm low, leaving the front-left
contact unloaded on straights: 1.6% -> 102.2% of demanded rolling.

None of them causes the left/right turn asymmetry, which survives all three.

Co-Authored-By: Claude Opus 5 <noreply@anthropic.com>
Claude-Session: https://claude.ai/code/session_01J91VAG6GU24wcgM3mWkjsN

File: picar2_description/urdf/picar2.urdf.xacro (robot description, xacro)
@@ -333,5 +333,5 @@
   <!-- Front wheels (passive — follow steer knuckle) -->
   <joint name="front_left_wheel_joint" type="continuous">
-    <origin xyz="0.00022897 0.0228 -0.0141" rpy="0 0 -0.010042"/>
+    <origin xyz="0.00022897 0.0228 -0.0137" rpy="0 0 -0.010042"/>   <!-- EXPERIMENT: front wheels coplanar with the rears -->
     <parent link="front_left_steer"/>
     <child  link="front_left_wheel"/>
@@ -344,12 +344,22 @@
          cannot exist. -->
     <axis xyz="0 1 0"/>
-    <dynamics damping="0.01" friction="0.0"/>
+    <!-- Passive wheels: essentially no bearing drag. At 0.01 the damping torque
+         is 0.10 N.m at driving speed (10 rad/s), while mu=0.5 on a 0.81 kg robot
+         supplies only 0.02-0.03 N.m to spin the wheel up - so the wheel could
+         sustain just 3.3 rad/s against the 10.6 the ground demands, and slid
+         instead of rolling. The outer wheel of a turn needs the higher rate, so
+         it stalled first and the stall swapped sides with the turn direction:
+         visible in Gazebo, and in the logs as the inner wheel rotating MORE than
+         the outer (left turn: front_left +53.4 rad against front_right +40.2).
+         The driven rear wheels keep 0.01 - their velocity controller overcomes
+         it. -->
+    <dynamics damping="0.0001" friction="0.0"/>
   </joint>
   <joint name="front_right_wheel_joint" type="continuous">
-    <origin xyz="-0.00025662 -0.019549 -0.0121" rpy="0 0 -0.013126"/>
+    <origin xyz="-0.00025662 -0.019549 -0.0117" rpy="0 0 -0.013126"/>   <!-- EXPERIMENT -->
     <parent link="front_right_steer"/>
     <child  link="front_right_wheel"/>
     <axis xyz="0 1 0"/>
-    <dynamics damping="0.01" friction="0.0"/>
+    <dynamics damping="0.0001" friction="0.0"/>   <!-- see front_left above -->
   </joint>
   <!-- Sensors (fixed) -->
