Commit message: sim: steer joint velocity 1.0 -> 4.0 rad/s, matching the real servo
gz_ros2_control's position mode hands DART a velocity command and DART
enforces the joint's velocity limit as a hard actuator cap; the real
Picar2Hardware path never reads this field at all (writes steer_delta_us
straight through the LUT). Step test (bare sim, cmd_vel step to 1.2):
every sim turn was throttled to a flat 59 deg/s (1.03 rad/s, exactly the
old limit) with no convergence curve - a third of the robot's measured
99th-pct 3.06 rad/s (bag obst_fix13_curvt20). Invalidates every prior sim
timing measurement of a swerve or corner. Fixed: 215 deg/s (3.75 rad/s)
against the new 4.0 limit.

Co-Authored-By: Claude Sonnet 5 <noreply@anthropic.com>
Claude-Session: https://claude.ai/code/session_01NACQRnKWkUxnf83R2Bsu1e

File: picar2_description/urdf/picar2.urdf.xacro (robot description, xacro)
@@ -320,5 +320,14 @@
     <dynamics damping="0.01" friction="0.0"/>
   </joint>
-  <!-- Front steering knuckles (revolute — single servo via linkage) -->
+  <!-- Front steering knuckles (revolute — single servo via linkage).
+       velocity=1 rad/s here throttled every sim turn to a third of the real
+       servo: Picar2Hardware writes steer_delta_us straight to the LUT and
+       never reads this field, but gz_ros2_control's position control mode
+       hands DART a velocity command and DART enforces this limit as a hard
+       actuator cap - a hard cap, not the shape of a real servo's response.
+       Step test (bare sim, cmd_vel step): the joint ramped at a dead-flat
+       59 deg/s (1.03 rad/s) into the stop, no convergence curve. Measured
+       on the robot (bag obst_fix13_curvt20): steering rate 99th pct 3.06
+       rad/s, peak 4.06. 4.0 leaves headroom without being make-believe. -->
   <joint name="front_left_steer_joint" type="revolute">
     <origin xyz="0.11922 0.065 0.0262" rpy="0 0 0"/>
@@ -326,5 +335,5 @@
     <child  link="front_left_steer"/>
     <axis xyz="0 0 1"/>
-    <limit lower="-0.6" upper="0.6" effort="10" velocity="1"/>
+    <limit lower="-0.6" upper="0.6" effort="10" velocity="4.0"/>
     <dynamics damping="0.01" friction="0.0"/>
   </joint>
@@ -334,5 +343,5 @@
     <child  link="front_right_steer"/>
     <axis xyz="0 0 1"/>
-    <limit lower="-0.6" upper="0.6" effort="10" velocity="1"/>
+    <limit lower="-0.6" upper="0.6" effort="10" velocity="4.0"/>
     <dynamics damping="0.01" friction="0.0"/>
   </joint>

Commit message: robot_model: per-chassis geometry for v1 and v2
Everything that follows the chassis moves out of the shared files into
picar2_description/models/<model>.yaml (xacro: axles, mounts, LUT) and
config/models/<model>/ (controllers/nav2 overlays, imu and mag calibration).
All launch files take robot_model:= (default v1); v1 output is unchanged,
v2 values are copies of v1 until measured, with its servo centre/limits.

Co-Authored-By: Claude Fable 5.1 <noreply@anthropic.com>
Claude-Session: https://claude.ai/code/session_01NACQRnKWkUxnf83R2Bsu1e

File: picar2_description/urdf/picar2.urdf.xacro (robot description, xacro)
@@ -5,4 +5,7 @@
   <xacro:arg name="use_sim" default="false"/>
   <xacro:arg name="lidar"   default="lds02rr"/>
+  <!-- Which chassis: models/<robot_model>.yaml holds every dimension, mount
+       and the steering LUT that differ between the robots. -->
+  <xacro:arg name="robot_model" default="v1"/>
   <!-- Scales every simulated sensor noise stddev. Gazebo Harmonic exposes no
        RNG seed, so sensor noise is the one source of run-to-run variance that
@@ -13,4 +16,6 @@
   <xacro:property name="noise_scale" value="$(arg sensor_noise)"/>
   <xacro:property name="lidar_model"    value="$(arg lidar)"/>
+  <xacro:property name="m" value="${xacro.load_yaml('$(find picar2_description)/models/$(arg robot_model).yaml')}"/>
+  <xacro:property name="lidar_mount" value="${m['lidar_mount'].get(lidar_model, m['lidar_mount']['default'])}"/>
   <xacro:property name="ld07_tilt_rad"  value="0.2793"/>  <!-- 16° mount angle -->
   <!-- ═══════════════════════════════════════════════════
@@ -27,9 +32,6 @@
         <param name="port">$(arg port)</param>
         <param name="baud">$(arg baud)</param>
-        <!-- Steering LUT: delta_us from servo center (ascending) and steer_rad in ROS convention
-             (positive = left turn, so positive deg measurement is negated here).
-             Measured 2026-05-22 from wheel-angle photo; refine with odom_cal circle test. -->
-        <param name="steer_lut_us">-595 -454 -410 -364 -329 -299 -271 -252 -202 -151 -121 -101 128 154	193	257	308	354	433	464	493	545</param>
-        <param name="steer_lut_rad">0.6756 0.5308 0.4578 0.4058 0.3513 0.3176 0.2790 0.2443 0.1994 0.1392 0.1062 0.0668 -0.1276 -0.1646 -0.2049 -0.2829	-0.3129	-0.3681	-0.4680	-0.4844	-0.5078	-0.6109</param>
+        <param name="steer_lut_us">${' '.join(map(str, m['steer_lut_us']))}</param>
+        <param name="steer_lut_rad">${' '.join(map(str, m['steer_lut_rad']))}</param>
         <!-- 30, not the driver's 50 default. The EKF runs at 50 Hz and is fed
              IMU at exactly its own rate with no headroom; on the robot it
@@ -98,4 +100,5 @@
               name="gz_ros2_control::GazeboSimROS2ControlPlugin">
         <parameters>$(find picar2_bringup)/config/controllers.yaml</parameters>
+        <parameters>$(find picar2_bringup)/config/models/$(arg robot_model)/controllers.yaml</parameters>
       </plugin>
       <!-- Ground-truth pose for the navigation benchmark. Simulation only, so
@@ -135,6 +138,6 @@
     </visual>
     <collision>
-      <origin xyz="0 0 0.04" rpy="0 0 0"/>
-      <geometry><box size="0.24 0.17 0.08"/></geometry>
+      <origin xyz="${m['chassis_collision']['xyz']}" rpy="0 0 0"/>
+      <geometry><box size="${m['chassis_collision']['size']}"/></geometry>
     </collision>
   </link>
@@ -154,5 +157,5 @@
     <collision>
       <origin xyz="0 0 0" rpy="1.5708 0 0"/>
-      <geometry><cylinder radius="0.033" length="0.025"/></geometry>
+      <geometry><cylinder radius="${m['wheel_radius']}" length="${m['wheel_width']}"/></geometry>
     </collision>
   </link>
@@ -172,5 +175,5 @@
     <collision>
       <origin xyz="0 0 0" rpy="1.5708 0 0"/>
-      <geometry><cylinder radius="0.033" length="0.025"/></geometry>
+      <geometry><cylinder radius="${m['wheel_radius']}" length="${m['wheel_width']}"/></geometry>
     </collision>
   </link>
@@ -208,5 +211,5 @@
     <collision>
       <origin xyz="0 0 0" rpy="1.5708 0 0"/>
-      <geometry><cylinder radius="0.033" length="0.025"/></geometry>
+      <geometry><cylinder radius="${m['wheel_radius']}" length="${m['wheel_width']}"/></geometry>
     </collision>
   </link>
@@ -244,5 +247,5 @@
     <collision>
       <origin xyz="0 0 0" rpy="1.5708 0 0"/>
-      <geometry><cylinder radius="0.033" length="0.025"/></geometry>
+      <geometry><cylinder radius="${m['wheel_radius']}" length="${m['wheel_width']}"/></geometry>
     </collision>
   </link>
@@ -298,14 +301,14 @@
     <parent link="base_footprint"/>
     <child  link="base_link"/>
-    <origin xyz="0.11607 0.0 0.0215" rpy="0 0 0"/>
+    <origin xyz="${m['base_link_xyz']}" rpy="0 0 0"/>
   </joint>
   <joint name="base_imu" type="fixed">
     <parent link="base_link"/>
     <child  link="imu_link"/>
-    <origin xyz="-0.05 0.0 0.05" rpy="0 0 0"/>
+    <origin xyz="${m['imu_xyz']}" rpy="0 0 0"/>
   </joint>
   <!-- Rear wheels (continuous — drive wheels) -->
   <joint name="back_right_joint" type="continuous">
-    <origin xyz="-0.11607 -0.08425 0.0125" rpy="0 0 0"/>
+    <origin xyz="${m['rear_right_xyz']}" rpy="0 0 0"/>
     <parent link="base_link"/>
     <child  link="back_right_link"/>
@@ -314,5 +317,5 @@
   </joint>
   <joint name="back_left_joint" type="continuous">
-    <origin xyz="-0.11607 0.08425 0.0125" rpy="0 0 0"/>
+    <origin xyz="${m['rear_left_xyz']}" rpy="0 0 0"/>
     <parent link="base_link"/>
     <child  link="back_left_link"/>
@@ -331,5 +334,5 @@
        rad/s, peak 4.06. 4.0 leaves headroom without being make-believe. -->
   <joint name="front_left_steer_joint" type="revolute">
-    <origin xyz="0.11922 0.065 0.0262" rpy="0 0 0"/>
+    <origin xyz="${m['steer_left_xyz']}" rpy="0 0 0"/>
     <parent link="base_link"/>
     <child  link="front_left_steer"/>
@@ -339,5 +342,5 @@
   </joint>
   <joint name="front_right_steer_joint" type="revolute">
-    <origin xyz="0.11922 -0.065 0.0242" rpy="0 0 0"/>
+    <origin xyz="${m['steer_right_xyz']}" rpy="0 0 0"/>
     <parent link="base_link"/>
     <child  link="front_right_steer"/>
@@ -348,5 +351,5 @@
   <!-- Front wheels (passive — follow steer knuckle) -->
   <joint name="front_left_wheel_joint" type="continuous">
-    <origin xyz="0.00022897 0.0228 -0.0137" rpy="0 0 -0.010042"/>   <!-- EXPERIMENT: front wheels coplanar with the rears -->
+    <origin xyz="${m['front_left_wheel']['xyz']}" rpy="${m['front_left_wheel']['rpy']}"/>   <!-- EXPERIMENT: front wheels coplanar with the rears -->
     <parent link="front_left_steer"/>
     <child  link="front_left_wheel"/>
@@ -372,5 +375,5 @@
   </joint>
   <joint name="front_right_wheel_joint" type="continuous">
-    <origin xyz="-0.00025662 -0.019549 -0.0117" rpy="0 0 -0.013126"/>   <!-- EXPERIMENT -->
+    <origin xyz="${m['front_right_wheel']['xyz']}" rpy="${m['front_right_wheel']['rpy']}"/>   <!-- EXPERIMENT -->
     <parent link="front_right_steer"/>
     <child  link="front_right_wheel"/>
@@ -380,15 +383,10 @@
   <!-- Sensors (fixed) -->
   <joint name="laser_joint" type="fixed">
-    <xacro:if value="${lidar_model == 'ld19'}">
-      <origin xyz="0.042548 0.005 0.127" rpy="0 0 0.0523605"/>
-    </xacro:if>
-    <xacro:unless value="${lidar_model == 'ld19'}">
-      <origin xyz="0.012548 0 0.127" rpy="0 0 0"/>
-    </xacro:unless>
+    <origin xyz="${lidar_mount['xyz']}" rpy="${lidar_mount['rpy']}"/>
     <parent link="base_link"/>
     <child  link="laser_link"/>
   </joint>
   <joint name="ld07_joint" type="fixed">
-    <origin xyz="0.172 0 0.034" rpy="0 ${ld07_tilt_rad} 0"/>
+    <origin xyz="${m['ld07_xyz']}" rpy="0 ${ld07_tilt_rad} 0"/>
     <parent link="base_link"/>
     <child  link="ld07_link"/>
@@ -397,5 +395,5 @@
   <link name="sen0628_link"/>
   <joint name="sen0628_joint" type="fixed">
-    <origin xyz="0.172 0 0.054" rpy="0 0 0"/>
+    <origin xyz="${m['sen0628_xyz']}" rpy="0 0 0"/>
     <parent link="base_link"/>
     <child  link="sen0628_link"/>
@@ -435,5 +433,5 @@
   </link>
   <joint name="pan_joint" type="revolute">
-    <origin xyz="0.14 0 0.065" rpy="0 0 0"/>
+    <origin xyz="${m['pan_xyz']}" rpy="0 0 0"/>
     <parent link="base_link"/>
     <child  link="pan_link"/>

Commit message: description: imu_rpy per model for the imu_link joint
The hardware interface remaps chip axes for the v1 board; a board that
carries the chip turned is expressed as a rotation in the model yaml.
v1 stays 0 0 0.

Co-Authored-By: Claude Fable 5.1 <noreply@anthropic.com>
Claude-Session: https://claude.ai/code/session_01NACQRnKWkUxnf83R2Bsu1e

File: picar2_description/urdf/picar2.urdf.xacro (robot description, xacro)
@@ -306,5 +306,5 @@
     <parent link="base_link"/>
     <child  link="imu_link"/>
-    <origin xyz="${m['imu_xyz']}" rpy="0 0 0"/>
+    <origin xyz="${m['imu_xyz']}" rpy="${m.get('imu_rpy', '0 0 0')}"/>
   </joint>
   <!-- Rear wheels (continuous — drive wheels) -->
